File: Hardware/PCB.brd (EAGLE design)
At the start: 170.2 x 111.3 mm, 103 parts, among them IC1 BD5229G-TR, IC4 XC6220A331MR-G, J1 FH34SRJ-24S-0.5SH_99_, J2 SAMACSYS_PARTS_USB4110-GF-A, J3 QWIIC_RIGHT_ANGLE, J4 112A-TAAR-R03_ATTEND, Q1 20V/4.2A/52mΩ/1.4W, Q2 20V/4.2A/52mΩ/1.4W, Q3 SI1308EDL-T1-GE3, U1 MCP73831, U2 ESP32-C6-WROOM-1-N8, U3 W25Q512JVEIQ, U4 MAX17048G+T10, U5 DS3231SN#

Commit message: Update Schematic and PCB
Parts:
- moved J2 0.22 mm to (168.0, 54.3)
- moved J3 0.10 mm to (165.2, 19.4)
Connections:
- removed net N$12: J2.B7
- net DN: now also J2.B7
Routing:
- net GND: track 700.7 -> 725.3 mm, vias 16 -> 17
- net EPD_CS: track 107.0 -> 128.5 mm
- net N$17: track 83.2 -> 64.6 mm
- net EPD_3V3: track 46.5 -> 64.3 mm, vias 5 -> 3
- net PREVGH: track 30.3 -> 16.0 mm
- net USB_D+: track 147.4 -> 135.8 mm, vias 2 -> 4
- net SCL: track 227.5 -> 216.3 mm
- net SDA: track 211.6 -> 202.7 mm
- net TX: track 129.3 -> 138.0 mm, vias 2 -> 0
- net EPD_3V3_C: track 100.2 -> 92.5 mm, vias 4 -> 3
- net SRC: track 25.8 -> 33.2 mm
- net N$16: track 140.4 -> 133.3 mm, vias 0 -> 2
- net IO/CHANGE: track 78.5 -> 72.0 mm
- net INT_RTC: track 120.0 -> 125.5 mm, vias 2 -> 4
- net PREVGL: track 35.8 -> 40.7 mm
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- added copper zone on layer 1, net GND
- added copper zone on layer 16, net GND
Other:
- board size 170.2 x 111.3 mm -> 170.2 x 111.2 mm
