File: Hardware/Schematic.sch (EAGLE design)
At the start: 103 parts, among them IC1 BD5229G-TR, IC4 XC6220A331MR-G, J1 FH34SRJ-24S-0.5SH_99_, J2 SAMACSYS_PARTS_USB4110-GF-A, J3 QWIIC_RIGHT_ANGLE, J4 112A-TAAR-R03_ATTEND, Q1 20V/4.2A/52mΩ/1.4W, Q2 20V/4.2A/52mΩ/1.4W, Q3 SI1308EDL-T1-GE3, U1 MCP73831, U2 ESP32-C6-WROOM-1-N8, U3 W25Q512JVEIQ, U4 MAX17048G+T10, U5 DS3231SN#

Commit message: Update Schematic and PCB
Connections:
- removed net N$12: J2.B7
- net DN: now also J2.B7
Other:
- moved on the sheet: EPD_C11
Changed lines of the file:
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@@
 <class number="0" name="default" width="0" drill="0">
+</class>
+<class number="1" name="New Class" width="0.3" drill="0">
 </class>
 </classes>
@@
 <attribute name="VALUE" x="-113.919" y="150.876" size="1.778" layer="96"/>
 </instance>
-<instance part="EPD_C11" gate="G$1" x="-104.14" y="149.86" smashed="yes" rot="R270">
-<attribute name="NAME" x="-103.759" y="150.876" size="1.778" layer="95"/>
-<attribute name="VALUE" x="-116.459" y="148.336" size="1.778" layer="96"/>
+<instance part="EPD_C11" gate="G$1" x="-106.68" y="149.86" smashed="yes" rot="R270">
+<attribute name="NAME" x="-106.299" y="150.876" size="1.778" layer="95"/>
+<attribute name="VALUE" x="-118.999" y="148.336" size="1.778" layer="96"/>
 </instance>
 <instance part="EPD_C10" gate="G$1" x="-93.98" y="147.32" smashed="yes" rot="R270">
@@
 </busses>
 <nets>
-<net name="VBUS" class="0">
+<net name="VBUS" class="1">
 <segment>
 <pinref part="PFMF.050.1" gate="G$1" pin="2"/>
@@
 </segment>
 </net>
-<net name="VUSB" class="0">
+<net name="VUSB" class="1">
 <segment>
 <pinref part="PFMF.050.1" gate="G$1" pin="1"/>
@@
 <wire x1="-121.92" y1="152.4" x2="-121.92" y2="154.94" width="0.1524" layer="91"/>
 <pinref part="SUPPLY28" gate="G$1" pin="GND"/>
-<pinref part="EPD_C11" gate="G$1" pin="2"/>
-<wire x1="-109.22" y1="149.86" x2="-121.92" y2="149.86" width="0.1524" layer="91"/>
-<wire x1="-121.92" y1="149.86" x2="-121.92" y2="152.4" width="0.1524" layer="91"/>
 <pinref part="EPD_C9" gate="G$1" pin="2"/>
 <wire x1="-114.3" y1="144.78" x2="-121.92" y2="144.78" width="0.1524" layer="91"/>
@@
 <pinref part="EPD_C10" gate="G$1" pin="2"/>
 <wire x1="-121.92" y1="147.32" x2="-121.92" y2="149.86" width="0.1524" layer="91"/>
+<wire x1="-121.92" y1="149.86" x2="-121.92" y2="152.4" width="0.1524" layer="91"/>
 <wire x1="-99.06" y1="147.32" x2="-121.92" y2="147.32" width="0.1524" layer="91"/>
 <pinref part="EPD_C7" gate="G$1" pin="2"/>
@@
 <wire x1="-121.92" y1="129.54" x2="-121.92" y2="137.16" width="0.1524" layer="91"/>
 <junction x="-121.92" y="152.4"/>
-<junction x="-121.92" y="149.86"/>
 <junction x="-121.92" y="144.78"/>
 <junction x="-121.92" y="147.32"/>
@@
 <junction x="-121.92" y="142.24"/>
 <junction x="-121.92" y="137.16"/>
+<pinref part="EPD_C11" gate="G$1" pin="2"/>
+<wire x1="-111.76" y1="149.86" x2="-121.92" y2="149.86" width="0.1524" layer="91"/>
+<junction x="-121.92" y="149.86"/>
 </segment>
 <segment>
@@
 <label x="-40.64" y="261.62" size="1.27" layer="94" rot="MR0" xref="yes"/>
 </segment>
-</net>
-<net name="N$12" class="0">
 <segment>
 <pinref part="J2" gate="G$1" pin="B7"/>
@@
 </segment>
 </net>
-<net name="EPD_3V3" class="0">
+<net name="EPD_3V3" class="1">
 <segment>
 <wire x1="-66.04" y1="193.04" x2="-68.58" y2="193.04" width="0.1524" layer="91"/>
@@
 <wire x1="-83.82" y1="149.86" x2="-91.44" y2="149.86" width="0.1524" layer="91"/>
 <pinref part="EPD_C11" gate="G$1" pin="1"/>
-<wire x1="-91.44" y1="149.86" x2="-101.6" y2="149.86" width="0.1524" layer="91"/>
+<wire x1="-91.44" y1="149.86" x2="-104.14" y2="149.86" width="0.1524" layer="91"/>
 <wire x1="-91.44" y1="149.86" x2="-91.44" y2="154.94" width="0.1524" layer="91"/>
 <label x="-91.44" y="154.94" size="1.27" layer="95" rot="R90" xref="yes"/>
@@
 <segment>
 <pinref part="EPD_C9" gate="G$1" pin="1"/>
-<wire x1="-83.82" y1="144.78" x2="-99.06" y2="144.78" width="0.1524" layer="91"/>
+<wire x1="-83.82" y1="144.78" x2="-101.6" y2="144.78" width="0.1524" layer="91"/>
 <pinref part="J1" gate="G$1" pin="21"/>
-<wire x1="-99.06" y1="144.78" x2="-106.68" y2="144.78" width="0.1524" layer="91"/>
-<wire x1="-99.06" y1="144.78" x2="-99.06" y2="154.94" width="0.1524" layer="91"/>
-<label x="-99.06" y="154.94" size="1.27" layer="95" rot="R90" xref="yes"/>
-<junction x="-99.06" y="144.78"/>
+<wire x1="-101.6" y1="144.78" x2="-106.68" y2="144.78" width="0.1524" layer="91"/>
+<wire x1="-101.6" y1="144.78" x2="-101.6" y2="154.94" width="0.1524" layer="91"/>
+<label x="-101.6" y="154.94" size="1.27" layer="95" rot="R90" xref="yes"/>
+<junction x="-101.6" y="144.78"/>
 </segment>
 </net>
@@
 </segment>
 </net>
-<net name="3V3" class="0">
+<net name="3V3" class="1">
 <segment>
 <pinref part="IC4" gate="G$1" pin="VOUT"/>
@@
 </segment>
 </net>
-<net name="EPD_3V3_C" class="0">
+<net name="EPD_3V3_C" class="1">
 <segment>
 <pinref part="U2" gate="G$1" pin="IO20"/>
@@
 <segment>
 <pinref part="IC1" gate="G$1" pin="VOUT"/>
-<wire x1="121.92" y1="121.92" x2="134.62" y2="121.92" width="0.1524" layer="91"/>
-<wire x1="134.62" y1="121.92" x2="139.7" y2="121.92" width="0.1524" layer="91"/>
-<junction x="134.62" y="121.92"/>
-<wire x1="134.62" y1="121.92" x2="134.62" y2="124.46" width="0.1524" layer="91"/>
+<wire x1="121.92" y1="121.92" x2="139.7" y2="121.92" width="0.1524" layer="91"/>
 <label x="139.7" y="121.92" size="1.27" layer="95" rot="R90" xref="yes"/>
 </segment>
@@
 <wire x1="134.62" y1="119.38" x2="139.7" y2="119.38" width="0.1524" layer="91"/>
 <pinref part="C5" gate="G$1" pin="1"/>
-<wire x1="134.62" y1="119.38" x2="134.62" y2="132.08" width="0.1524" layer="91"/>
+<junction x="134.62" y="119.38"/>
 <pinref part="R_RESET" gate="G$1" pin="2"/>
-<junction x="134.62" y="119.38"/>
-</segment>
-</net>
+<wire x1="134.62" y1="132.08" x2="134.62" y2="119.38" width="0.1524" layer="91"/>
+</segment>
+</net>
