File: Hardware/Schematic.sch (EAGLE design)
At the start: 103 parts, among them IC1 BD5229G-TR, IC4 XC6220A331MR-G, J1 FH34SRJ-24S-0.5SH_99_, J2 SAMACSYS_PARTS_USB4110-GF-A, J3 QWIIC_RIGHT_ANGLE, J4 112A-TAAR-R03_ATTEND, Q1 20V/4.2A/52mΩ/1.4W, Q2 20V/4.2A/52mΩ/1.4W, Q3 SI1308EDL-T1-GE3, U1 MCP73831, U2 ESP32-C6-WROOM-1-N8, U3 W25Q512JVEIQ, U4 MAX17048G+T10, U5 DS3231SN#

Commit message: Solve schematic issue
Connections:
- removed net N$18: C5.1, RESET_BUTTON.3, RESET_BUTTON.4, R_RESET.2
- removed net N$8: SENSOR2.CSB, SENSOR2.VDD
- net I2C_PW: now also SENSOR2.CSB, SENSOR2.VDD
- net RESET: now also C5.1, RESET_BUTTON.3, RESET_BUTTON.4, R_RESET.2
Changed lines of the file:
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@@
 </segment>
 <segment>
+<pinref part="SENSOR2" gate="G$1" pin="CSB"/>
+<wire x1="12.7" y1="144.78" x2="10.16" y2="144.78" width="0.1524" layer="91"/>
+<wire x1="10.16" y1="144.78" x2="10.16" y2="160.02" width="0.1524" layer="91"/>
+<wire x1="10.16" y1="160.02" x2="45.72" y2="160.02" width="0.1524" layer="91"/>
+<wire x1="43.18" y1="149.86" x2="45.72" y2="149.86" width="0.1524" layer="91"/>
+<pinref part="SENSOR2" gate="G$1" pin="VDD"/>
+<wire x1="45.72" y1="149.86" x2="45.72" y2="152.4" width="0.1524" layer="91"/>
+<wire x1="50.8" y1="154.94" x2="50.8" y2="152.4" width="0.1524" layer="91"/>
+<wire x1="50.8" y1="152.4" x2="45.72" y2="152.4" width="0.1524" layer="91"/>
 <pinref part="SENSOR2" gate="G$1" pin="VDDIO"/>
-<wire x1="43.18" y1="152.4" x2="50.8" y2="152.4" width="0.1524" layer="91"/>
-<wire x1="50.8" y1="152.4" x2="50.8" y2="154.94" width="0.1524" layer="91"/>
 <label x="50.8" y="154.94" size="1.27" layer="95" rot="R90" xref="yes"/>
+<wire x1="45.72" y1="152.4" x2="43.18" y2="152.4" width="0.1524" layer="91"/>
+<junction x="45.72" y="152.4"/>
+<wire x1="45.72" y1="152.4" x2="45.72" y2="160.02" width="0.1524" layer="91"/>
 </segment>
 <segment>
@@
 <segment>
 <pinref part="IC1" gate="G$1" pin="VOUT"/>
-<wire x1="121.92" y1="121.92" x2="139.7" y2="121.92" width="0.1524" layer="91"/>
+<wire x1="121.92" y1="121.92" x2="134.62" y2="121.92" width="0.1524" layer="91"/>
 <label x="139.7" y="121.92" size="1.27" layer="95" rot="R90" xref="yes"/>
+<pinref part="R_RESET" gate="G$1" pin="2"/>
+<wire x1="134.62" y1="121.92" x2="139.7" y2="121.92" width="0.1524" layer="91"/>
+<wire x1="134.62" y1="132.08" x2="134.62" y2="121.92" width="0.1524" layer="91"/>
+<junction x="134.62" y="121.92"/>
+<pinref part="RESET_BUTTON" gate="G$1" pin="3"/>
+<wire x1="132.08" y1="119.38" x2="134.62" y2="119.38" width="0.1524" layer="91"/>
+<pinref part="RESET_BUTTON" gate="G$1" pin="4"/>
+<wire x1="134.62" y1="119.38" x2="139.7" y2="119.38" width="0.1524" layer="91"/>
+<junction x="134.62" y="119.38"/>
+<pinref part="C5" gate="G$1" pin="1"/>
+<wire x1="134.62" y1="119.38" x2="134.62" y2="121.92" width="0.1524" layer="91"/>
 </segment>
 </net>
@@
 </segment>
 </net>
-<net name="N$8" class="0">
-<segment>
-<pinref part="SENSOR2" gate="G$1" pin="CSB"/>
-<wire x1="12.7" y1="144.78" x2="10.16" y2="144.78" width="0.1524" layer="91"/>
-<wire x1="10.16" y1="144.78" x2="10.16" y2="160.02" width="0.1524" layer="91"/>
-<wire x1="10.16" y1="160.02" x2="45.72" y2="160.02" width="0.1524" layer="91"/>
-<wire x1="45.72" y1="160.02" x2="45.72" y2="149.86" width="0.1524" layer="91"/>
-<wire x1="45.72" y1="149.86" x2="43.18" y2="149.86" width="0.1524" layer="91"/>
-<pinref part="SENSOR2" gate="G$1" pin="VDD"/>
-</segment>
-</net>
 <net name="N$9" class="0">
 <segment>
@@
 </segment>
 </net>
-<net name="N$18" class="0">
-<segment>
-<pinref part="RESET_BUTTON" gate="G$1" pin="3"/>
-<wire x1="132.08" y1="119.38" x2="134.62" y2="119.38" width="0.1524" layer="91"/>
-<pinref part="RESET_BUTTON" gate="G$1" pin="4"/>
-<wire x1="134.62" y1="119.38" x2="139.7" y2="119.38" width="0.1524" layer="91"/>
-<junction x="134.62" y="119.38"/>
-<wire x1="134.62" y1="132.08" x2="134.62" y2="119.38" width="0.1524" layer="91"/>
-<pinref part="R_RESET" gate="G$1" pin="2"/>
-<pinref part="C5" gate="G$1" pin="1"/>
-</segment>
-</net>
